File: PDB_12V/ODOS_PDB_12V_schem.kicad_sch (KiCad schematic)
At the start: 8 parts, among them J1 XT30UPB-F, J2 XT30UPB-F, J3 XT30UPB-F, J4 XT30UPB-F, J5 XT30UPB-F, J6 XT30UPB-F

Commit message: nouveau layout et 2 plans pour gnd et +12
Parts:
- added C2: 820µF, Capacitor_SMD:CP_Elec_10x10.5, symbol Device:C_Polarized
Connections:
- net +12V: now also J1.2 (P), J2.2 (P), J3.2 (P), J4.2 (P), J5.2 (P), J6.2 (P), C2.1; no longer J1.1 (P), J2.1 (P), J3.1 (P), J4.1 (P), J5.1 (P), J6.1 (P)
- net GND: now also J1.1 (N), J2.1 (N), J3.1 (N), J4.1 (N), J5.1 (N), J6.1 (N), C2.2; no longer J1.2 (N), J2.2 (N), J3.2 (N), J4.2 (N), J5.2 (N), J6.2 (N)
Other:
- moved on the sheet: J6
